File: schematics/main_schematic.sch (EAGLE design)
At the start: 42 parts, among them Q1 IRLML0030TRPBF, Q2 IRLML0030TRPBF, Q3 IRLML0030TRPBF

Commit message: Schematic converted to hierarchical layout
Parts:
- removed C1, C2, C3, C4, C5, C6: 100nF, resistor:C-EUC0805
- removed C7, C8: (no value), resistor:C-EUC0805
- removed FAN1: FAN1, Rembrandt Electronics - JST XH Connectors v1-0:JST-XH-03-PIN-LONG-PAD
- removed FAN2: FAN2, Rembrandt Electronics - JST XH Connectors v1-0:JST-XH-03-PIN-LONG-PAD
- removed FAN3: FAN3, Rembrandt Electronics - JST XH Connectors v1-0:JST-XH-03-PIN-LONG-PAD
- removed JP1: FAN2_Vcc, jumper:JP3QE
- removed JP2: FAN1_Vcc, jumper:JP3QE
- removed JP3: FAN3_Vcc, jumper:JP3QE
- removed LED1, LED2, LED3: (no value), led:LEDSMT1206
- removed Q1, Q2, Q3: IRLML0030TRPBF, fets:MOSFET-NCHANNELSMD
- removed R1, R12, R15, R2, R3, R4, R5, R6, R9: 10K, resistor:R-EU_R0805
- removed R10, R13, R7: 2K7, resistor:R-EU_R0805
- removed R11, R14, R8: 100R, resistor:R-EU_R0805
- removed U$1: DUE(NORMAL), DUElib130425:DUE(NORMAL)
- removed XMAX: X-MAX, Rembrandt Electronics - JST XH Connectors v1-0:JST-XH-03-PIN-LONG-PAD
- removed XMIN: X-MIN, Rembrandt Electronics - JST XH Connectors v1-0:JST-XH-03-PIN-LONG-PAD
- removed YMAX: Y-MAX, Rembrandt Electronics - JST XH Connectors v1-0:JST-XH-03-PIN-LONG-PAD
- removed YMIN: Y-MIN, Rembrandt Electronics - JST XH Connectors v1-0:JST-XH-03-PIN-LONG-PAD
- removed ZMAX: Z-MAX, Rembrandt Electronics - JST XH Connectors v1-0:JST-XH-03-PIN-LONG-PAD
- removed ZMIN: Z-MIN, Rembrandt Electronics - JST XH Connectors v1-0:JST-XH-03-PIN-LONG-PAD
Connections:
- removed net +12V: JP1-2.1, JP2-2.1, JP3-2.1, U$1.VIN
- removed net +24V: JP1-1.1, JP2-1.1, JP3-1.1
- removed net +3V3: U$1.3V3, U$1.IOREF
- removed net +5V: C7.1, C8.1, JP1-3.1, JP2-3.1, JP3-3.1, U$1.5V, U$1.GND_ICSP, XMAX-2.S, XMIN-2.S, YMAX-2.S, YMIN-2.S, ZMAX-2.S, ZMIN-2.S
- removed net 25: U$1.25
- removed net 27: U$1.27
- removed net 29: U$1.29
- removed net 31: U$1.31
- removed net 33: U$1.33
- removed net 35: U$1.35
- removed net 37: U$1.37
- removed net BED: U$1.39
- removed net BEEPER: U$1.41
- removed net CANRX: U$1.CANRX
- removed net CANTX: U$1.CANTX
- removed net CARDDETECT: U$1.TX3
- removed net CS0: U$1.10
- removed net CS1: U$1.4
- removed net DAC0: U$1.DAC0
- removed net DAC1: U$1.DAC1
- removed net E1-DIR: U$1.53
- removed net E1-ENA: U$1.A11
- removed net E1-STP: U$1.51
- removed net E2-DIR: U$1.23
- removed net E2-ENA: U$1.49
- removed net E2-STP: U$1.24
- removed net ENCA: U$1.52
- removed net ENCB: U$1.50
- removed net ENCP: U$1.48
- removed net FAN1: R8.1, U$1.11
- removed net FAN1+: FAN1-2.S, JP2-1.2, JP2-2.2, JP2-3.2, R7.1
- removed net FAN1-: FAN1-3.S, LED1.C, Q1.D
- removed net FAN2: R11.1, U$1.9
- removed net FAN2+: FAN2-2.S, JP1-1.2, JP1-2.2, JP1-3.2, R10.1
- removed net FAN2-: FAN2-3.S, LED2.C, Q2.D
- removed net FAN3: R14.1, U$1.12
- removed net FAN3+: FAN3-2.S, JP3-1.2, JP3-2.2, JP3-3.2, R13.1
- removed net FAN3-: FAN3-3.S, LED3.C, Q3.D
- removed net GND: C1.2, C2.2, C3.2, C4.2, C5.2, C6.2, C7.2, C8.2, Q1.S, Q2.S, Q3.S, R12.2, R15.2, R9.2, U$1.5V_ICSP, U$1.GND_1, U$1.GND_2, XMAX-1.S, XMIN-1.S, YMAX-1.S, YMIN-1.S, ZMAX-1.S, ZMIN-1.S
- removed net HOT1: U$1.8
- removed net HOT2: U$1.7
- removed net LCD4: U$1.44
- removed net LCD5: U$1.45
- removed net LCD6: U$1.46
- removed net LCD7: U$1.47
- removed net LCD_ENA: U$1.43
- removed net LCD_RS: U$1.42
- removed net MISO: U$1.MISO_ICSP
- removed net MOSI: U$1.MOSI_ICSP
- removed net N$1: LED3.A, R13.2
- removed net N$2: LED1.A, R7.2
- removed net N$3: LED2.A, R10.2
- removed net N$4: Q2.G, R11.2, R12.1
- removed net N$5: Q1.G, R8.2, R9.1
- removed net N$6: Q3.G, R14.2, R15.1
- removed net NTC1: U$1.A0
- removed net NTC2: U$1.A1
- removed net NTC3: U$1.A2
- removed net NTC4: U$1.A5
- removed net PSON: U$1.40
- removed net PWM1: U$1.5
- removed net PWM2: U$1.6
- removed net PWM3: U$1.13
- removed net RESET: U$1.RESET_ICSP
- removed net RX0: U$1.RX0
- removed net RX1: U$1.RX1
- removed net SCK: U$1.SCK_ICSP
- removed net SCL: U$1.SCL
- removed net SCL1: U$1.SCL1
- removed net SDA: U$1.SDA
- removed net SDA1: U$1.SDA1
- removed net TC-K1: U$1.A4
- removed net TC-K2: U$1.A3
- removed net TX0: U$1.TX0
- removed net TX1: U$1.TX1
- removed net X-DIR: U$1.3
- removed net X-ENA: U$1.22
- removed net X-MAX: C2.1, R2.2, U$1.36
- removed net X-MAX-OUT: R2.1, XMAX-3.S
- removed net X-MIN: C1.1, R1.2, U$1.38
- removed net X-MIN-OUT: R1.1, XMIN-3.S
- removed net X-STP: U$1.2
- removed net Y-DIR: U$1.TX2
- removed net Y-ENA: U$1.26
- removed net Y-MAX: C4.1, R4.2, U$1.32
- removed net Y-MAX-OUT: R4.1, YMAX-3.S
- removed net Y-MIN: C3.1, R3.2, U$1.34
- removed net Y-MIN-OUT: R3.1, YMIN-3.S
- removed net Y-STP: U$1.RX2
- removed net Z-MAX: C6.1, R6.2, U$1.28
- removed net Z-MAX-OUT: R6.1, ZMAX-3.S
- removed net Z-MIN: C5.1, R5.2, U$1.30
- removed net Z-MIN-OUT: R5.1, ZMIN-3.S
- removed net Z1-DIR: U$1.A6
- removed net Z1-ENA: U$1.RX3
- removed net Z1-STP: U$1.A7
- removed net Z2-DIR: U$1.A9
- removed net Z2-ENA: U$1.A8
- removed net Z2-STP: U$1.A10
