File: schematics/main_schematic.brd (EAGLE design)
At the start: 252.7 x 134.3 mm, 128 parts

Commit message: Working on PCB
Parts:
- added HEATBED:J2, HOTEND1:J2, HOTEND2:J2: (no value), SparkFun-Connectors:SCREWTERMINAL-5MM-2
- E1:C11, E2:C11, X:C11, Y:C11, Z1:C11, Z2:C11: device resistor:PANASONIC_B -> rcl:PANASONIC_D
- moved RESET:S1 430.4 mm to (143.1, 6.60), turned to 180 degrees
- moved RESET:X1 426.5 mm to (146.8, 16.4), turned to 90 degrees
- moved HC-POWER-SUPPLY-HOTEND:J2 389.9 mm to (146.3, 91.4), turned to 90 degrees
- moved EXP2:EXP2 371.7 mm to (92.2, 118.6), turned to 90 degrees
- moved EXP1:EXP1 356.1 mm to (83.3, 118.6), turned to 90 degrees
- moved HC-POWER-SUPPLY-HOTEND:F1 356.0 mm to (126.0, 98.6), turned to 180 degrees
- moved TERM3:X1 329.2 mm to (42.4, 112.9), turned to 90 degrees
- moved HC-POWER-SUPPLY-HEATBED:J2 327.9 mm to (146.3, 121.9), turned to 90 degrees
- moved HOTEND2:R3 325.8 mm to (117.1, 65.0), turned to 180 degrees
- moved HOTEND2:LED1 320.4 mm to (108.7, 74.7)
- moved HC-POWER-SUPPLY:J2 315.3 mm to (146.3, 137.2), turned to 90 degrees
- moved HOTEND2:R2 309.8 mm to (117.1, 74.7), turned to 180 degrees
- moved HOTEND2:Q1 302.1 mm to (124.5, 69.8), turned to 270 degrees
- moved TERM4:X1 299.6 mm to (42.4, 123.1), turned to 90 degrees
- moved HOTEND2:R1 299.5 mm to (112.8, 74.7)
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Connections:
- new net HEATBED:N$4: HEATBED:J2.1, HEATBED:Q1.C
- new net HOTEND1:N$4: HOTEND1:J2.1, HOTEND1:Q1.C
- new net HOTEND2:N$4: HOTEND2:J2.1, HOTEND2:Q1.C
- net N$63: now also HOTEND1:J2.2, HOTEND2:J2.2; no longer HOTEND1:Q1.C, HOTEND2:Q1.C
- net N$67: now also HEATBED:J2.2; no longer HEATBED:Q1.C
Other:
- board size 252.7 x 134.3 mm -> 150 x 150 mm
